File: iot-plug.kicad_sch (KiCad schematic)
At the start: 32 parts, among them J1 Conn_01x02_Pin, J1 USB_C_Receptacle_USB2.0_16P, J2 Conn_01x02_Pin, K1 HF46F_005-HS1, Q2 2N3904, U1 ESP32-S3-MINI-1, U1 USBLC6-2SC6, U4 AMS1117-3.3

Commit message: layout updated
Parts:
- renumbered J1 to J3, U1 to U2
Changed lines of the file:
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@@
 (kicad_sch
-	(version 20231120)
+	(version 20250114)
 	(generator "eeschema")
-	(generator_version "8.0")
+	(generator_version "9.0")
 	(paper "A4")
+	(rectangle
+		(start 94.488 95.758)
+		(end 106.68 144.526)
+		(stroke
+			(width 0)
+			(type default)
+		)
+		(fill
+			(type none)
+		)
+	)
+	(rectangle
+		(start 105.664 156.464)
+		(end 173.99 193.294)
+		(stroke
+			(width 0)
+			(type default)
+		)
+		(fill
+			(type none)
+		)
+	)
+	(rectangle
+		(start 16.002 96.012)
+		(end 52.832 144.78)
+		(stroke
+			(width 0)
+			(type default)
+		)
+		(fill
+			(type none)
+		)
+	)
+	(rectangle
+		(start 14.986 156.464)
+		(end 102.87 193.294)
+		(stroke
+			(width 0)
+			(type default)
+		)
+		(fill
+			(type none)
+		)
+	)
+	(rectangle
+		(start 14.986 16.002)
+		(end 77.724 85.09)
+		(stroke
+			(width 0)
+			(type default)
+		)
+		(fill
+			(type none)
+		)
+	)
+	(rectangle
+		(start 54.356 95.758)
+		(end 92.964 144.526)
+		(stroke
+			(width 0)
+			(type default)
+		)
+		(fill
+			(type none)
+		)
+	)
+	(text "3V3-LDO"
+		(exclude_from_sim no)
+		(at 118.11 160.782 0)
+		(effects
+			(font
+				(size 3.048 3.048)
+				(thickness 0.254)
+				(bold yes)
+			)
+		)
+	)
+	(text "TypeC-Uart"
+		(exclude_from_sim no)
+		(at 61.722 80.772 0)
+		(effects
+			(font
+				(size 3.048 3.048)
+				(thickness 0.254)
+				(bold yes)
+			)
+		)
+	)
 	(junction
 		(at 34.29 104.14)
@@
 		)
 	)
-	(rectangle
-		(start 94.488 95.758)
-		(end 106.68 144.526)
-		(stroke
-			(width 0)
-			(type default)
-		)
-		(fill
-			(type none)
-		)
-	)
-	(rectangle
-		(start 105.664 156.464)
-		(end 173.99 193.294)
-		(stroke
-			(width 0)
-			(type default)
-		)
-		(fill
-			(type none)
-		)
-	)
-	(rectangle
-		(start 16.002 96.012)
-		(end 52.832 144.78)
-		(stroke
-			(width 0)
-			(type default)
-		)
-		(fill
-			(type none)
-		)
-	)
-	(rectangle
-		(start 14.986 156.464)
-		(end 102.87 193.294)
-		(stroke
-			(width 0)
-			(type default)
-		)
-		(fill
-			(type none)
-		)
-	)
-	(rectangle
-		(start 14.986 16.002)
-		(end 77.724 85.09)
-		(stroke
-			(width 0)
-			(type default)
-		)
-		(fill
-			(type none)
-		)
-	)
-	(rectangle
-		(start 54.356 95.758)
-		(end 92.964 144.526)
-		(stroke
-			(width 0)
-			(type default)
-		)
-		(fill
-			(type none)
-		)
-	)
-	(text "3V3-LDO"
-		(exclude_from_sim no)
-		(at 118.11 160.782 0)
-		(effects
-			(font
-				(size 3.048 3.048)
-				(thickness 0.254)
-				(bold yes)
-			)
-		)
-	)
-	(text "TypeC-Uart"
-		(exclude_from_sim no)
-		(at 61.722 80.772 0)
-		(effects
-			(font
-				(size 3.048 3.048)
-				(thickness 0.254)
-				(bold yes)
-			)
-		)
-	)
 	(label "IO1"
 		(at 101.6 104.14 270)
-		(fields_autoplaced yes)
 		(effects
 			(font
@@
 	(label "N"
 		(at 68.58 140.97 180)
-		(fields_autoplaced yes)
 		(effects
 			(font
@@
 	(label "D-"
 		(at 48.26 45.72 0)
-		(fields_autoplaced yes)
 		(effects
 			(font
@@
 	(label "D+"
 		(at 256.54 53.34 180)
-		(fields_autoplaced yes)
 		(effects
 			(font
@@
 	(label "IO1"
 		(at 256.54 63.5 180)
-		(fields_autoplaced yes)
 		(effects
 			(font
@@
 	(label "EN"
 		(at 34.29 99.06 270)
-		(fields_autoplaced yes)
 		(effects
 			(font
@@
 	(label "P"
 		(at 86.36 139.7 180)
-		(fields_autoplaced yes)
 		(effects
 			(font
@@
 	(label "N"
 		(at 24.13 175.26 180)
-		(fields_autoplaced yes)
 		(effects
 			(font
@@
 	(label "D+"
 		(at 69.85 50.8 180)
-		(fields_autoplaced yes)
 		(effects
 			(font
@@
 	(label "D-"
 		(at 256.54 55.88 180)
-		(fields_autoplaced yes)
 		(effects
 			(font
@@
 	(label "D-"
 		(at 69.85 48.26 180)
-		(fields_autoplaced yes)
 		(effects
 			(font
@@
 	(label "P"
 		(at 24.13 170.18 0)
-		(fields_autoplaced yes)
 		(effects
 			(font
@@
 	(label "IO0"
 		(at 256.54 60.96 180)
-		(fields_autoplaced yes)
 		(effects
 			(font
@@
 	(label "D+"
 		(at 48.26 50.8 0)
-		(fields_autoplaced yes)
 		(effects
 			(font
@@
 	(label "EN"
 		(at 157.48 45.72 0)
-		(fields_autoplaced yes)
 		(effects
 			(font
@@
 	(label "IO0"
 		(at 34.29 123.19 270)
-		(fields_autoplaced yes)
 		(effects
 			(font
@@
 		(on_board yes)
 		(dnp no)
-		(property "Reference" "U1"
+		(property "Reference" "U2"
 			(at 61.214 55.118 0)
 			(effects
@@
 		(on_board yes)
 		(dnp no)
-		(property "Reference" "#PWR01"
+		(property "Reference" "#PWR0101"
 			(at 25.4 78.74 0)
 			(effects
@@
 		(on_board yes)
 		(dnp no)
-		(property "Reference" "J1"
+		(property "Reference" "J3"
 			(at 21.082 28.956 90)
 			(effects
@@
 		)
 	)
+	(embedded_fonts no)
 )

Commit message: updated tracks & nets
Connections:
- net RL: now also U1.25 (GPIO21)
Other:
- note added: "AC-DC"
- note added: "Buttons"
- note added: "Led"
- note added: "Relay"
- moved on the sheet: C1, C6, C7, D2, D6, EN1, F1, H1, J1, J2, K1, PRG1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
